File: PCB/Split keyboard.kicad_pcb (KiCad board)
At the start: 2 copper layers, 312.4 x 114 mm, 125 parts, among them SW1 SW_SPDT, SW10 SW_Push, SW11 SW_Push, SW12 SW_Push, SW13 SW_Push, SW14 SW_Push, SW15 SW_Push, SW16 SW_Push, SW17 SW_Push, SW18 SW_Push, SW19 SW_Push, SW2 SW_Push, SW20 SW_Push, SW21 SW_Push, SW22 SW_Push, SW23 SW_Push, SW24 SW_Push, SW25 SW_Push, SW26 SW_Push, SW27 SW_Push, SW28 SW_Push, SW29 SW_Push, SW3 SW_Push, SW30 SW_Push, SW31 SW_Push, SW32 SW_Push, SW33 SW_Push, SW34 SW_Push, SW35 SW_Push, SW36 SW_Push, SW37 SW_Push, SW38 SW_Push, SW39 SW_Push, SW4 SW_Push, SW40 SW_Push, SW41 SW_Push, SW42 SW_Push, SW43 SW_Push, SW44 SW_SPDT, SW47 SW_Push, SW48 SW_Push, SW49 SW_Push, SW5 SW_Push, SW50 SW_Push, SW6 SW_Push, SW7 SW_Push, SW8 SW_Push, SW9 SW_Push, U1 XIAO-nRF52840-SMD, U2 XIAO-nRF52840-SMD, U3 74HC165

Commit message: Updated Joystick footprint to THT and added BOM
Parts:
- JS1: footprint PCM_marbastlib-xp-various:PNT_psp1000 -> Connector_PinHeader_2.54mm:PinHeader_1x04_P2.54mm_Vertical
- moved JS1 8.48 mm to (185.8, 111.8)
Routing:
- net GND: track 151.2 -> 123.2 mm, vias 25 -> 21
- net /right_half/JOY_X: track 124.4 -> 139.7 mm
- net /right_half/JOY_Y: track 145.6 -> 158.5 mm, vias 0 -> 1
- net /right_half/3V3: track 134.2 -> 144.8 mm, vias 10 -> 11
- net Net-(D31-DOUT): track 81.5 -> 86.4 mm

Commit message: pcb
Routing:
- net /right_half/3V3: vias 11 -> 10
Changed lines of the file:
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@@
+	)
+	(segment
+		(start 188.547214 116.622786)
+		(end 185.75 119.42)
+		(width 0.5)
+		(layer "F.Cu")
+		(net 71)
 	)
 	(segment
@@
 	)
 	(segment
-		(start 188.525 110.011214)
-		(end 188.525 114.825)
-		(width 0.2)
+		(start 188.547214 109.989)
+		(end 188.547214 116.622786)
+		(width 0.5)
 		(layer "F.Cu")
 		(net 71)
@@
 	)
 	(via
-		(at 188.525 114.825)
-		(size 0.6)
-		(drill 0.3)
-		(layers "F.Cu" "B.Cu")
-		(net 71)
-	)
-	(via
 		(at 281.93 91.03)
 		(size 0.6)
@@
 	)
 	(segment
-		(start 188.525 116.645)
-		(end 185.75 119.42)
-		(width 0.2)
-		(layer "B.Cu")
-		(net 71)
-	)
-	(segment
 		(start 220.28 101.86)
 		(end 237.24 101.86)
@@
 		(layer "B.Cu")
 		(net 71)
-	)
-	(segment
-		(start 188.525 114.825)
-		(end 188.525 116.645)
-		(width 0.2)
-		(layer "B.Cu")
-		(net 71)
